File: LaserCo2Board/LaserCo2Board.sch (KiCad schematic (older format))
At the start: 99 parts, among them J1 Y VREF, J10 Y1 MOTOR, J11 Y2 MOTOR, J12 USB, J13 X LIMIT, J14 Y LIMIT, J15 D SWITCH, J2 X VREF, J3 LASER, J4 POWER IN, J6 PCB FAN, J7 BOX FAN, J8 JTAG, J9 X MOTOR, SW1 SW_PUSH, SW2 SWITCH_INV, U1 STM32F20XR, U2 A4982SLPTR, U3 A4982SLPTR, U4 74VHC1GT08, U5 74HC1G00, U6 MCP44X1, U7 LD1117S33TR, X1 CRYSTAL_4PIN, X2 CRYSTAL

Commit message: First Commit
Parts:
- added L2: BLM21PG221SN1D, ~, symbol FILTER
- added PTC1: MF-MSMF050-2 500mA, ~, symbol THERMISTOR
- added VR1, VR2: CG0603MLC-05E, ~, symbol VR
Connections:
- wire segments 422 -> 432
Other:
- moved on the sheet: C32, J12, R28, R29

Commit message: First Commit
Parts:
- removed J3: LASER, ~, symbol CONN5
- removed J4: POWER IN, ~, symbol CONN3
- removed PTC1: MF-MSMF050-2 500mA, ~, symbol THERMISTOR
- removed U4: 74VHC1GT08, ~, symbol 74HC1G08
- added C27, C28, C38: 0u1, symbol C_SMALL
- added C37: 10u, symbol C_SMALL
- added D4: X2 Stop, symbol LED
- added D5: Y2 Stop, symbol LED
- added J10: LASER, ~, symbol CONN3
- added J13: WATER FLOW, ~, symbol CONN3
- added J15: LASER P, ~, symbol CONN2
- added J17: X LIMIT2, ~, symbol CONN2
- added J19: Y LIMIT2, ~, symbol CONN2
- added J5: POWER IN, ~, symbol CONN2
- added J8: FAN3, ~, symbol CONN2
- added J9: PUMP, ~, symbol CONN2
- added Q1, Q2, Q3: BSS138, ~, symbol MOSFET_N
- added R23, R24, R27, R29, R30, R33, R37, R38: 10k, symbol R
- added R25, R26: 470R, symbol R
- added R34: 75R, symbol R
- added R35: 1k5, symbol R
- added R36: 390R, symbol R
- added U5: 74HC08A, ~, symbol 74HC08A
- added U6: MCP4725, ~, symbol MCP4725
- D1: value Y Stop -> X1 Stop
- D2: value Z Stop -> Y1 Stop
- D3: value E1 Stop -> D Stop
- J16: renamed from J13; value X LIMIT -> X LIMIT1
- J18: renamed from J14; value Y LIMIT -> Y LIMIT1
- J6: value PCB FAN -> FAN1
- J7: value BOX FAN -> FAN2
- renumbered C24 to C22, C26 to C23, C27 to C24, C29 to C25, C22 to C26, C23 to C29, C25 to C31, C31 to C32, C28 to C33, C32 to C35, C33 to C36, D4 to D6, D5 to D7, D6 to D8, J9 to J11, J10 to J12, J11 to J14, J15 to J20, J8 to J3, J12 to J4, R32 to R1, R9 to R10, R10 to R11, R11 to R12, R12 to R13, R13 to R14, R14 to R15, R15 to R16, R16 to R17, R17 to R18, R22 to R19, R1 to R2, R23 to R20, R24 to R21, R25 to R22, R18 to R28, R2 to R3, R19 to R31, R20 to R32, R28 to R39, R3 to R4, R29 to R40, R21 to R41, R26 to R42, R27 to R43, R30 to R44, R31 to R45, R4 to R5, R5 to R6, R6 to R7, R7 to R8, R8 to R9, U7 to U4, U6 to U7, U5 to U8
Connections:
- net labels added: CHECK_12V, LASER_ANALOG, LASER_POINT, LASER_POINT_CONN, SCL1, SDA1, WATER_FLOW, X_LIMIT1, X_LIMIT2, X_LIMIT_CONN1, X_LIMIT_CONN2, Y_LIMIT1, Y_LIMIT2, Y_LIMIT_CONN1, Y_LIMIT_CONN2
- net labels removed: X_LIMIT, X_LIMIT_CONN, Y_LIMIT, Y_LIMIT_CONN
- wire segments 432 -> 521
- no-connect marks 38 -> 32
Other:
- note added: "12V Input"
- note added: "5V Output"
- note added: "Analog Output"
- note added: "Endstops"
- note removed: "Endstops."
- moved on the sheet: C15, C16, C17, C18, C19, C20, C22, C24, C26, C29, C30, C31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

Commit message: First Commit
Parts:
- added C39: 100u, symbol C_POL
Connections:
- wire segments 521 -> 523
Other:
- moved on the sheet: J8, J9
Changed lines of the file:
@@
 Sheet 1 1
 Title "LaserCo2Board"
-Date "29 aug 2016"
+Date "30 aug 2016"
 Rev "1.0.0"
 Comp "smartDIYs Co.,Ltd."
@@
 L CONN2 J8
 U 1 1 57C28AD8
-P 16400 2600
-F 0 "J8" H 16400 2500 40  0000 C CNN
-F 1 "FAN3" V 16550 2650 40  0000 C CNN
-F 2 "~" H 16400 2600 60  0000 C CNN
-F 3 "~" H 16400 2600 60  0000 C CNN
-	1    16400 2600
+P 16400 2700
+F 0 "J8" H 16400 2600 40  0000 C CNN
+F 1 "FAN3" V 16550 2750 40  0000 C CNN
+F 2 "~" H 16400 2700 60  0000 C CNN
+F 3 "~" H 16400 2700 60  0000 C CNN
+	1    16400 2700
 	1    0    0    -1
 $EndComp
@@
 L GND #PWR044
 U 1 1 57C28ADE
-P 15550 2700
-F 0 "#PWR044" H 15550 2700 30  0001 C CNN
-F 1 "GND" H 15550 2630 30  0001 C CNN
-F 2 "" H 15550 2700 60  0001 C CNN
-F 3 "" H 15550 2700 60  0001 C CNN
-	1    15550 2700
+P 15550 2900
+F 0 "#PWR044" H 15550 2900 30  0001 C CNN
+F 1 "GND" H 15550 2830 30  0001 C CNN
+F 2 "" H 15550 2900 60  0001 C CNN
+F 3 "" H 15550 2900 60  0001 C CNN
+	1    15550 2900
 	1    0    0    -1
 $EndComp
-Text GLabel 15900 2500 0    60   Input ~ 0
+Text GLabel 15650 2550 0    60   Input ~ 0
 V_IN
 Wire Wire Line
-	16050 2600 15550 2600
+	15550 2750 15550 2900
 Wire Wire Line
-	15550 2600 15550 2700
-Wire Wire Line
-	15900 2500 16050 2500
+	15650 2550 16050 2550
 $Comp
 L CONN2 J9
 U 1 1 57C28AE8
-P 16400 2950
-F 0 "J9" H 16400 2850 40  0000 C CNN
-F 1 "PUMP" V 16550 3000 40  0000 C CNN
-F 2 "~" H 16400 2950 60  0000 C CNN
-F 3 "~" H 16400 2950 60  0000 C CNN
-	1    16400 2950
+P 16400 3200
+F 0 "J9" H 16400 3100 40  0000 C CNN
+F 1 "PUMP" V 16550 3250 40  0000 C CNN
+F 2 "~" H 16400 3200 60  0000 C CNN
+F 3 "~" H 16400 3200 60  0000 C CNN
+	1    16400 3200
 	1    0    0    -1
 $EndComp
@@
 L GND #PWR045
 U 1 1 57C28AEE
-P 15550 3050
-F 0 "#PWR045" H 15550 3050 30  0001 C CNN
-F 1 "GND" H 15550 2980 30  0001 C CNN
-F 2 "" H 15550 3050 60  0001 C CNN
-F 3 "" H 15550 3050 60  0001 C CNN
-	1    15550 3050
+P 15550 3300
+F 0 "#PWR045" H 15550 3300 30  0001 C CNN
+F 1 "GND" H 15550 3230 30  0001 C CNN
+F 2 "" H 15550 3300 60  0001 C CNN
+F 3 "" H 15550 3300 60  0001 C CNN
+	1    15550 3300
 	1    0    0    -1
 $EndComp
-Text GLabel 15900 2850 0    60   Input ~ 0
+Text GLabel 15900 3100 0    60   Input ~ 0
 V_IN
 Wire Wire Line
-	16050 2950 15550 2950
+	16050 3200 15550 3200
 Wire Wire Line
-	15550 2950 15550 3050
+	15550 3200 15550 3300
 Wire Wire Line
-	15900 2850 16050 2850
+	15900 3100 16050 3100
 Wire Notes Line
 	15150 4150 15150 3750
@@
 Wire Wire Line
 	10050 9450 10200 9450
+$Comp
+L C_POL C39
+U 1 1 57C500C9
+P 15800 2650
+F 0 "C39" H 15750 2800 50  0000 L CNN
+F 1 "100u" H 15850 2600 50  0000 L CNN
+F 2 "" H 15800 2650 60  0001 C CNN
+F 3 "" H 15800 2650 60  0001 C CNN
+	1    15800 2650
+	1    0    0    -1
+$EndComp
+Wire Wire Line
+	16050 2550 16050 2600
+Connection ~ 15800 2550
+Wire Wire Line
+	15550 2750 16050 2750
+Wire Wire Line
+	16050 2750 16050 2700
+Connection ~ 15800 2750
 $EndSCHEMATC

Commit message: サンプル確認後の修正
#16
#15
#14
#13
#12
Parts:
- removed Q2: BSS138, ~, symbol MOSFET_N
- removed R33: 10k, symbol R
- added TR2: BSH105, ~, symbol BSH105
- R27: value 10k -> 100R
- R34: value 75R -> 22R
- R44: value 1K -> 1k5
- renumbered Q3 to Q2
Connections:
- wire segments 523 -> 521
Other:
- moved on the sheet: C39, J7, R1, R34

Commit message: 変更
Parts:
- removed R27: 100R, symbol R
- removed TR2: BSH105, ~, symbol BSH105
- R34: value 22R -> 47R
Connections:
- net labels removed: LASER_POINT, LASER_POINT_CONN
- wire segments 521 -> 515
- no-connect marks 32 -> 33
Other:
- note removed: "5V Output"
- moved on the sheet: R34
Changed lines of the file:
@@
 Sheet 1 1
 Title "LaserCo2Board"
-Date "27 sep 2016"
+Date "5 oct 2016"
 Rev "1.0.0"
 Comp "smartDIYs Co.,Ltd."
@@
 Text GLabel 1100 12400 1    39   Input ~ 0
 CHECK_12V
-Text GLabel 1100 13800 0    39   Output ~ 0
-LASER_POINT
 $Comp
 L GND #PWR035
@@
 NoConn ~ 11550 1950
 NoConn ~ 11550 1850
-Text GLabel 10250 12000 0    39   Output ~ 0
-LASER_POINT
 $Comp
 L GND #PWR037
@@
 L R R34
 U 1 1 57C29F42
-P 11450 11300
-F 0 "R34" V 11530 11300 50  0000 C CNN
-F 1 "22R" V 11450 11300 50  0000 C CNN
-F 2 "" H 11450 11300 60  0001 C CNN
-F 3 "" H 11450 11300 60  0001 C CNN
-	1    11450 11300
-	1    0    0    -1
+P 19400 3650
+F 0 "R34" V 19480 3650 50  0000 C CNN
+F 1 "47R" V 19400 3650 50  0000 C CNN
+F 2 "" H 19400 3650 60  0001 C CNN
+F 3 "" H 19400 3650 60  0001 C CNN
+	1    19400 3650
+	0    -1   -1   0
 $EndComp
 Text GLabel 11500 9800 0    39   Input ~ 0
@@
 Text GLabel 12400 10000 2    39   Input ~ 0
 CHECK_12V
-Text GLabel 11450 10950 1    39   Input ~ 0
+Text GLabel 19050 3650 0    39   Input ~ 0
 VBUS
-Text GLabel 11700 11600 2    39   Output ~ 0
-LASER_POINT_CONN
 $Comp
 L CONN2 J15
@@
 	1    0    0    -1
 $EndComp
-Text GLabel 19550 3650 0    60   Input ~ 0
-LASER_POINT_CONN
 $Comp
 L CONN2 J17
@@
 Text GLabel 19700 2050 0    60   Input ~ 0
 Y_LIMIT_CONN2
-Text Notes 9850 10900 0    60   ~ 0
-5V Output
 Text GLabel 11550 13150 1    60   Input ~ 0
 SDA1
@@
 $EndComp
 NoConn ~ 1350 13700
-$Comp
-L BSH105 TR2
-U 1 1 57E9DFA1
-P 11300 12000
-F 0 "TR2" H 11203 12250 70  0000 C CNN
-F 1 "BSH105" H 11153 11703 60  0000 C CNN
-F 2 "~" H 11300 12000 60  0000 C CNN
-F 3 "~" H 11300 12000 60  0000 C CNN
-	1    11300 12000
-	1    0    0    -1
-$EndComp
-$Comp
-L R R27
-U 1 1 57E9DFB5
-P 10600 12000
-F 0 "R27" V 10680 12000 50  0000 C CNN
-F 1 "100R" V 10500 12000 50  0000 C CNN
-F 2 "" H 10600 12000 60  0001 C CNN
-F 3 "" H 10600 12000 60  0001 C CNN
-	1    10600 12000
-	0    1    1    0
-$EndComp
-$Comp
-L GND #PWR045
-U 1 1 57E9DFEE
-P 11450 12400
-F 0 "#PWR045" H 11450 12400 30  0001 C CNN
-F 1 "GND" H 11450 12330 30  0001 C CNN
-F 2 "" H 11450 12400 60  0001 C CNN
-F 3 "" H 11450 12400 60  0001 C CNN
-	1    11450 12400
-	1    0    0    -1
-$EndComp
 Wire Notes Line
 	13750 8600 13750 6450
@@
 	1100 13600 1350 13600
 Wire Wire Line
-	1100 13800 1350 13800
-Wire Wire Line
 	9000 3700 9000 3900
 Connection ~ 9000 5050
@@
 	15150 4200 20900 4200
 Wire Wire Line
-	19550 3650 19750 3650
-Wire Wire Line
 	19750 3750 19600 3750
 Wire Wire Line
@@
 	20150 2450 19700 2450
 Wire Wire Line
-	11450 11600 11700 11600
-Wire Wire Line
 	10050 13150 10050 13450
 Wire Wire Line
@@
 	9750 12600 9900 12600
 Wire Notes Line
-	9750 10700 12550 10700
-Wire Notes Line
-	12550 10700 12550 12500
-Wire Notes Line
-	12550 12500 9750 12500
-Wire Notes Line
-	9750 12500 9750 10700
-Wire Notes Line
 	11300 9450 12900 9450
 Wire Notes Line
@@
 	1100 12500 1100 12400
 Wire Wire Line
-	11450 10950 11450 11050
-Wire Wire Line
-	11450 11550 11450 11650
-Wire Wire Line
-	11450 12350 11450 12400
-Wire Wire Line
-	11000 12000 10850 12000
-Wire Wire Line
-	10350 12000 10250 12000
-Connection ~ 11450 11600
+	19050 3650 19150 3650
 NoConn ~ 1350 12800
 NoConn ~ 1350 12900
@@
 Wire Wire Line
 	15900 2650 16050 2650
+NoConn ~ 1350 13800
+Wire Wire Line
+	19650 3650 19750 3650
 $EndSCHEMATC

Commit message: ノイズ対策
Parts:
- added C40: 0u1, symbol C_SMALL
- added L3, L4: BLM21SN300SN1D, ~, symbol FILTER
- added R27: 22R, symbol R_SMALL
- U2: footprint (none) -> ~
Connections:
- net labels added: LASER_OUT_CONN
- wire segments 515 -> 532
Other:
- moved on the sheet: C39, J11, J5

Commit message: ノイズ対策2
Parts:
- removed C37: 10u, symbol C_SMALL
- removed Q1, Q2: BSS138, ~, symbol MOSFET_N
- removed R27: 22R, symbol R_SMALL
- removed R29, R30, R37, R38: 10k, symbol R
- added C41, C43: 10u, ~, symbol CP1
- added C42: 0u1, symbol C_SMALL
- added L5: inductor, ~, symbol INDUCTOR
- added R27: 220R, symbol R
- added R29, R30, R37, R38: 4k7, symbol R_SMALL
- added R33: 1k, symbol R
- added U10: IB0505S, symbol IB0505S
- added U11: ADUM1250, symbol ADUM1250
- added U9: TLP2355, ~, symbol TLP2355
Connections:
- net labels added: D5V, DGND
- wire segments 532 -> 556
Other:
- moved on the sheet: C32, C34, C35, C36, C38, C39, D6, D7, D8, J10, J11, J12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

Commit message: 元に戻す
Parts:
- removed C41, C43: 10u, ~, symbol CP1
- removed C42: 0u1, symbol C_SMALL
- removed L5: inductor, ~, symbol INDUCTOR
- removed R27: 220R, symbol R
- removed R29, R30, R37, R38: 4k7, symbol R_SMALL
- removed R33: 1k, symbol R
- removed U10: IB0505S, symbol IB0505S
- removed U11: ADUM1250, symbol ADUM1250
- removed U9: TLP2355, ~, symbol TLP2355
- added C37: 10u, symbol C_SMALL
- added Q1, Q2: BSS138, ~, symbol MOSFET_N
- added R27: 22R, symbol R_SMALL
- added R29, R30, R37, R38: 10k, symbol R
Connections:
- net labels removed: D5V, DGND
- wire segments 556 -> 532
Other:
- moved on the sheet: C32, C34, C35, C36, C38, C39, D6, D7, D8, J10, J11, J12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
